Commit message: final phase commit

File: src/my_robot_description/urdf/mobile_base.xacro (robot description, xacro)
@@ -5,5 +5,5 @@
     <xacro:property name="base_height" value="0.2"/>
     <xacro:property name="wheel_length" value="0.08"/>
-   <link name="base_footprint"/>
+    <link name="base_footprint"/>
     <link name="base_link">
         <visual>
@@ -28,9 +28,8 @@
         </collision>
     </link>
-    <xacro:macro name="wheel_link" params="prefix">
-    <link name="${prefix}_wheel_link">
+    <link name="front_left_wheel">
             <visual>
                 <geometry>
-                    <cylinder radius="0.125" length="0.08"/>
+                    <cylinder radius="0.27" length="0.08"/>
                 </geometry>
                 <origin xyz="0 0 0" rpy="${pi/ 2.0} 0 0"/>
@@ -39,42 +38,41 @@
             <collision>
                 <geometry>
-                    <cylinder radius="0.125" length="0.08"/>
+                    <cylinder radius="0.27" length="0.08"/>
                 </geometry>
                 <origin xyz="0 0 0" rpy="${pi/ 2.0} 0 0"/>
             </collision>
-            <xacro:cylinder_inertia m="10" r="0.1" h="0.05" xyz="0 0 0" rpy="${pi/ 2.0} 0 0"/>
-        </link>
-    </xacro:macro>
-    <xacro:wheel_link prefix="right_front"/>
-    <xacro:wheel_link prefix="left_front"/>
-    <xacro:wheel_link prefix="right_back"/>
-    <xacro:wheel_link prefix="left_back"/>
+            <xacro:cylinder_inertia m="10" r="0.27" h="0.05" xyz="0 0 0" rpy="${pi/ 2.0} 0 0"/>
+    </link>
+    <link name="front_right_wheel">
+            <visual>
+                <geometry>
+                    <cylinder radius="0.27" length="0.08"/>
+                </geometry>
+                <origin xyz="0 0 0" rpy="${pi/ 2.0} 0 0"/>
+                <material name="grey"/>
+            </visual>
+            <collision>
+                <geometry>
+                    <cylinder radius="0.27" length="0.08"/>
+                </geometry>
+                <origin xyz="0 0 0" rpy="${pi/ 2.0} 0 0"/>
+            </collision>
+            <xacro:cylinder_inertia m="10" r="0.27" h="0.05" xyz="0 0 0" rpy="${pi/ 2.0} 0 0"/>
+    </link>
     <joint name="base_footprint_link" type="fixed">
         <parent link="base_footprint"/>
         <child link="base_link"/>
-        <origin xyz="0 0 0" rpy="0 0 0"/>
+        <origin xyz="0 0 0.08" rpy="0 0 0"/>
     </joint>
-    <joint name="base_right_front_wheel_joint" type="continuous">
+    <joint name="right_wheel_joint" type="continuous">
         <parent link="base_link"/>
-        <child link="right_front_wheel_link"/>
-        <origin xyz="-0.255  ${-(base_width/ 2.0) - 0.03} 0.125" rpy="0 0 0"/>
+        <child link="front_right_wheel"/>
+        <origin xyz="0  ${-(base_width/ 2.0) - 0.05} 0.19" rpy="0 0 0"/>
         <axis xyz="0 1 0"/>
     </joint>
-    <joint name="base_left_front_wheel_joint" type="continuous">
+    <joint name="left_wheel_joint" type="continuous">
         <parent link="base_link"/>
-        <child link="left_front_wheel_link"/>
-        <origin xyz="0.255  ${(base_width / 2.0) + 0.03} 0.125" rpy="0 0 0"/>
-        <axis xyz="0 1 0"/>
-    </joint>
-        <joint name="base_right_back_wheel_joint" type="continuous">
-        <parent link="base_link"/>
-        <child link="right_back_wheel_link"/>
-        <origin xyz="0.225  ${-(base_width/ 2.0) - 0.03} 0.125" rpy="0 0 0"/>
-        <axis xyz="0 1 0"/>
-    </joint>
-    <joint name="base_left_back_wheel_joint" type="continuous">
-        <parent link="base_link"/>
-        <child link="left_back_wheel_link"/>
-        <origin xyz="-0.225  ${(base_width / 2.0) + 0.03} 0.125" rpy="0 0 0"/>
+        <child link="front_left_wheel"/>
+        <origin xyz="0  ${(base_width / 2.0) + 0.05} 0.19" rpy="0 0 0"/>
         <axis xyz="0 1 0"/>
     </joint>

File: src/my_robot_description/urdf/my_robot.urdf.xacro (robot description, xacro)
@@ -3,5 +3,4 @@
     <xacro:include filename="common_properties.xacro"/>
     <xacro:include filename="mobile_base.xacro"/>
-    <xacro:include filename="mobile_base_gazebo.xacro"/>
     <xacro:include filename="rover_platform.xacro"/>
     <xacro:include filename="rover_sensors.xacro"/>

File: src/my_robot_description/urdf/rover_sensors.xacro (robot description, xacro)
@@ -10,5 +10,5 @@
         </visual>
     </link>
-    <link name="camera_front">
+    <link name="front_camera">
         <visual>
             <geometry>
@@ -58,7 +58,12 @@
     <joint name="camera_front_platform_joint" type="fixed">
         <parent link="horizontal_camera_stand" />
-        <child link="camera_front" />
+        <child link="front_camera" />
         <origin xyz="0.075 0 0" rpy="0 0 0"/>
     </joint>
+    <!-- <joint name="camera_front_joint" type="fixed">
+        <parent link="front_camera" />
+        <child link="zed_camera_link" />
+        <origin xyz="0.075 0 0" rpy="0 0 0"/>
+    </joint> -->
     <joint name="camera_back_platform_joint" type="fixed">
         <parent link="horizontal_camera_stand" />
